Commit message: Started manually correcting poppy ergo jr urdf transformations

File: pybullet/poppy_ergo_jr/data/poppy_ergo_jr.urdf (robot description, URDF)
Before this commit: robot PoppyErgoJr, 7 links, 6 joints
Links:
- removed link section_2
- removed link section_3
- removed link section_4
- removed link tip
- link section_1: geometry collision mesh filename=PoppyErgoJr/meshes/horn2horn.stl; visual mesh filename=PoppyErgoJr/meshes/horn2horn.stl
Joints:
- removed joint m3
- removed joint m4
- removed joint m5
- removed joint m6
- joint m1: origin xyz=0 0 0.0327993216120967 rpy=-6.12303176911189E-17 0 0 -> xyz=0 0 25 rpy=0 0 0
- joint m2: origin xyz=0 0 0.0240006783879033 rpy=1.5707963267949 0 0 -> xyz=0 0 25 rpy=0 0 0
