Commit message: urdf tweaks and angle transforms from real poppy to pybullet

File: urdfs/humanoid/poppy_humanoid.urdf (robot description, URDF)
Before this commit: robot Poppy_Humanoid, 26 links, 25 joints
Joints:
- joint bust_y: limit lower=-1.16937059884 upper=0.471238898038 effort=3.1 velocity=7.0 -> lower=-0.471238898038 upper=1.16937059884 effort=3.1 velocity=7.0
- joint head_y: limit lower=-0.785398163397 upper=0.10471975512 effort=1.8 velocity=10.0 -> lower=-0.10471975512 upper=0.785398163397 effort=1.8 velocity=10.0
- joint l_hip_x: limit lower=-0.523598775598 upper=0.497418836818 effort=3.1 velocity=7.0 -> lower=-0.497418836818 upper=0.523598775598 effort=3.1 velocity=7.0
- joint l_hip_z: limit lower=-0.436332312999 upper=1.57079632679 effort=3.1 velocity=7.0 -> lower=-1.57079632679 upper=0.436332312999 effort=3.1 velocity=7.0
- joint l_knee_y: limit lower=-0.0610865238198 upper=2.33874119767 effort=3.1 velocity=7.0 -> lower=-2.33874119767 upper=0.0610865238198 effort=3.1 velocity=7.0
- joint l_shoulder_x: limit lower=-1.83259571459 upper=1.91986217719 effort=3.1 velocity=7.0 -> lower=-1.91986217719 upper=1.83259571459 effort=3.1 velocity=7.0
- joint r_hip_x: limit lower=-0.497418836818 upper=0.523598775598 effort=3.1 velocity=7.0 -> lower=-0.523598775598 upper=0.497418836818 effort=3.1 velocity=7.0
- joint r_hip_z: limit lower=-1.57079632679 upper=0.436332312999 effort=3.1 velocity=7.0 -> lower=-0.436332312999 upper=1.57079632679 effort=3.1 velocity=7.0
- joint r_shoulder_x: limit lower=-1.91986217719 upper=1.83259571459 effort=3.1 velocity=7.0 -> lower=-1.83259571459 upper=1.91986217719 effort=3.1 velocity=7.0
- joint r_shoulder_y: limit lower=-2.70526034059 upper=2.09439510239 effort=3.1 velocity=7.0 -> lower=-2.09439510239 upper=2.70526034059 effort=3.1 velocity=7.0
