Commit message: progress on ori.urdf correction

File: urdfs/humanoid/poppy_humanoid.ori.urdf (robot description, URDF)
Before this commit: robot Poppy_Humanoid, 26 links, 25 joints
Joints:
- joint abs_y: axis -1 0 0 -> 1 0 0
- joint bust_y: axis -1 0 0 -> 1 0 0
- joint l_hip_x: axis 0 0 -1 -> 0 0 1
- joint l_knee_y: axis 0 0 -1 -> 0 0 1
- joint l_shoulder_x: axis 0 0 1 -> 0 0 -1; origin xyz=0.0284 0 0 rpy=3.14159265358979 0 1.5707963267949 -> xyz=0.0284 0 0 rpy=3.14159265358979 0 0
- joint l_shoulder_y: origin xyz=0.0771000000000001 0.0499999999999999 0.00399999999999997 rpy=-1.5707963267949 0 0 -> xyz=0.0771000000000001 0.0499999999999999 0.00399999999999997 rpy=0 0 0
- joint r_hip_x: axis 0 0 -1 -> 0 0 1
- joint r_knee_y: axis 0 0 -1 -> 0 0 1
- joint r_shoulder_x: origin xyz=-0.0284 0 0 rpy=3.14159265358979 0 -1.5707963267949 -> xyz=-0.0284 0 0 rpy=3.14159265358979 0 0
- joint r_shoulder_y: axis -1 0 0 -> 1 0 0; origin xyz=-0.0770999999999999 0.0500000000000002 0.00400000000000003 rpy=-1.5707963267949 0 0 -> xyz=-0.0770999999999999 0.0500000000000002 0.00400000000000003 rpy=0 0 0

Commit message: ori.urdf good except for legs

File: urdfs/humanoid/poppy_humanoid.ori.urdf (robot description, URDF)
Before this commit: robot Poppy_Humanoid, 26 links, 25 joints
Joints:
- joint head_y: axis -1 0 0 -> 1 0 0
- joint l_arm_z: axis 0 1 0 -> 0 -1 0
- joint r_arm_z: axis 0 1 0 -> 0 -1 0
- joint r_elbow_y: axis -1 0 0 -> 1 0 0
