Commit message: reorganized pybullet envs, need to polish urdf search path in humanoid env

File: urdfs/humanoid/poppy_humanoid.pybullet.urdf (robot description, URDF)
Before this commit: robot Poppy_Humanoid, 26 links, 25 joints
Joints:
- joint l_hip_x: limit lower=-0.523598775598 upper=0.497418836818 effort=3.1 velocity=7.0 -> lower=-0.497418836818 upper=0.523598775598 effort=3.1 velocity=7.0
- joint l_hip_z: limit lower=-0.436332312999 upper=1.57079632679 effort=3.1 velocity=7.0 -> lower=-1.57079632679 upper=0.436332312999 effort=3.1 velocity=7.0
- joint l_knee_y: limit lower=-0.0610865238198 upper=2.33874119767 effort=3.1 velocity=7.0 -> lower=-2.33874119767 upper=0.0610865238198 effort=3.1 velocity=7.0
- joint l_shoulder_x: limit lower=-1.83259571459 upper=1.91986217719 effort=3.1 velocity=7.0 -> lower=-1.91986217719 upper=1.83259571459 effort=3.1 velocity=7.0

File: urdfs/humanoid/poppy_humanoid.urdf (robot description, URDF)
Before this commit: robot Poppy_Humanoid, 26 links, 25 joints
Joints:
- joint l_hip_x: limit lower=-0.497418836818 upper=0.523598775598 effort=3.1 velocity=7.0 -> lower=-0.523598775598 upper=0.497418836818 effort=3.1 velocity=7.0
- joint l_hip_z: limit lower=-1.57079632679 upper=0.436332312999 effort=3.1 velocity=7.0 -> lower=-0.436332312999 upper=1.57079632679 effort=3.1 velocity=7.0
- joint l_knee_y: limit lower=-2.33874119767 upper=0.0610865238198 effort=3.1 velocity=7.0 -> lower=-0.0610865238198 upper=2.33874119767 effort=3.1 velocity=7.0
- joint l_shoulder_x: limit lower=-1.91986217719 upper=1.83259571459 effort=3.1 velocity=7.0 -> lower=-1.83259571459 upper=1.91986217719 effort=3.1 velocity=7.0

Commit message: all angles fixed in poppy_humanoid.pybullet.urdf

File: urdfs/humanoid/poppy_humanoid.pybullet.urdf (robot description, URDF)
Before this commit: robot Poppy_Humanoid, 26 links, 25 joints
Joints:
- joint abs_y: axis -1 0 0 -> 1 0 0
- joint bust_y: axis -1 0 0 -> 1 0 0
- joint head_y: axis -1 0 0 -> 1 0 0
- joint l_arm_z: axis 0 1 0 -> 0 -1 0
- joint l_hip_x: axis 0 0 -1 -> 0 0 1; limit lower=-0.497418836818 upper=0.523598775598 effort=3.1 velocity=7.0 -> lower=-0.523598775598 upper=0.497418836818 effort=3.1 velocity=7.0
- joint l_hip_z: axis 0 -1 0 -> 0 1 0; limit lower=-1.57079632679 upper=0.436332312999 effort=3.1 velocity=7.0 -> lower=-0.436332312999 upper=1.57079632679 effort=3.1 velocity=7.0
- joint l_knee_y: axis 0 0 -1 -> 0 0 1; limit lower=-2.33874119767 upper=0.0610865238198 effort=3.1 velocity=7.0 -> lower=-0.0610865238198 upper=2.33874119767 effort=3.1 velocity=7.0
- joint l_shoulder_x: axis 0 0 1 -> 0 0 -1; limit lower=-1.91986217719 upper=1.83259571459 effort=3.1 velocity=7.0 -> lower=-1.83259571459 upper=1.91986217719 effort=3.1 velocity=7.0; origin xyz=0.0284 0 0 rpy=3.14159265358979 0 1.5707963267949 -> xyz=0.0284 0 0 rpy=3.14159265358979 0 0
- joint l_shoulder_y: origin xyz=0.0771000000000001 0.0499999999999999 0.00399999999999997 rpy=-1.5707963267949 0 0 -> xyz=0.0771000000000001 0.0499999999999999 0.00399999999999997 rpy=0 0 0
- joint r_ankle_y: axis -1 0 0 -> 1 0 0
- joint r_arm_z: axis 0 1 0 -> 0 -1 0
- joint r_elbow_y: axis -1 0 0 -> 1 0 0
- joint r_hip_x: axis 0 0 -1 -> 0 0 1
- joint r_hip_y: axis -1 0 0 -> 1 0 0
- joint r_hip_z: axis 0 -1 0 -> 0 1 0
- joint r_knee_y: axis 0 0 -1 -> 0 0 1
- joint r_shoulder_x: origin xyz=-0.0284 0 0 rpy=3.14159265358979 0 -1.5707963267949 -> xyz=-0.0284 0 0 rpy=3.14159265358979 0 0
- joint r_shoulder_y: axis -1 0 0 -> 1 0 0; origin xyz=-0.0770999999999999 0.0500000000000002 0.00400000000000003 rpy=-1.5707963267949 0 0 -> xyz=-0.0770999999999999 0.0500000000000002 0.00400000000000003 rpy=0 0 0

Commit message: fixed upper/lower limits for changed rotation axes in poppy_humanoid.pybullet.urdf

File: urdfs/humanoid/poppy_humanoid.pybullet.urdf (robot description, URDF)
Before this commit: robot Poppy_Humanoid, 26 links, 25 joints
Joints:
- joint abs_y: limit lower=-0.872664625997 upper=0.209439510239 effort=7.3 velocity=8.2 -> lower=-0.209439510239 upper=0.872664625997 effort=7.3 velocity=8.2
- joint bust_y: limit lower=-1.16937059884 upper=0.471238898038 effort=3.1 velocity=7.0 -> lower=-0.471238898038 upper=1.16937059884 effort=3.1 velocity=7.0
- joint head_y: limit lower=-0.785398163397 upper=0.10471975512 effort=1.8 velocity=10.0 -> lower=-0.10471975512 upper=0.785398163397 effort=1.8 velocity=10.0
- joint l_hip_x: limit lower=-0.523598775598 upper=0.497418836818 effort=3.1 velocity=7.0 -> lower=-0.497418836818 upper=0.523598775598 effort=3.1 velocity=7.0
- joint l_hip_z: limit lower=-0.436332312999 upper=1.57079632679 effort=3.1 velocity=7.0 -> lower=-1.57079632679 upper=0.436332312999 effort=3.1 velocity=7.0
- joint l_shoulder_x: limit lower=-1.83259571459 upper=1.91986217719 effort=3.1 velocity=7.0 -> lower=-1.91986217719 upper=1.83259571459 effort=3.1 velocity=7.0
- joint r_elbow_y: limit lower=-0.0174532925199 upper=2.58308729295 effort=3.1 velocity=7.0 -> lower=-2.58308729295 upper=0.0174532925199 effort=3.1 velocity=7.0
- joint r_hip_x: limit lower=-0.497418836818 upper=0.523598775598 effort=3.1 velocity=7.0 -> lower=-0.523598775598 upper=0.497418836818 effort=3.1 velocity=7.0
- joint r_hip_y: limit lower=-1.4835298642 upper=1.83259571459 effort=7.3 velocity=8.2 -> lower=-1.83259571459 upper=1.4835298642 effort=7.3 velocity=8.2
- joint r_hip_z: limit lower=-1.57079632679 upper=0.436332312999 effort=3.1 velocity=7.0 -> lower=-0.436332312999 upper=1.57079632679 effort=3.1 velocity=7.0
- joint r_knee_y: limit lower=-2.33874119767 upper=0.0610865238198 effort=3.1 velocity=7.0 -> lower=-0.0610865238198 upper=2.33874119767 effort=3.1 velocity=7.0
- joint r_shoulder_y: limit lower=-2.70526034059 upper=2.09439510239 effort=3.1 velocity=7.0 -> lower=-2.09439510239 upper=2.70526034059 effort=3.1 velocity=7.0

Commit message: all checked but l_shoulder_y

File: urdfs/humanoid/poppy_humanoid.pybullet.urdf (robot description, URDF)
Before this commit: robot Poppy_Humanoid, 26 links, 25 joints
Joints:
- joint l_shoulder_y: limit lower=-2.09439510239 upper=2.70526034059 effort=3.1 velocity=7.0 -> lower=-4.1887902047863905 upper=1.0471975511965976 effort=3.1 velocity=7.0
- joint r_shoulder_x: limit lower=-1.91986217719 upper=1.83259571459 effort=3.1 velocity=7.0 -> lower=-3.3335788713091694 upper=0.2792526803190927 effort=3.1 velocity=7.0
- joint r_shoulder_y: limit lower=-2.09439510239 upper=2.70526034059 effort=3.1 velocity=7.0 -> lower=-4.171336912266447 upper=1.0821041362364843 effort=3.1 velocity=7.0
