Commit message: basic pick and place cubes working

File: urdfs/objects/cube.urdf (robot description, URDF)
Before this commit: robot cube, 1 links, 0 joints
Links:
- removed link cube
- added link base_link, mass 1.2; collision box size=0.02 0.02 0.02; visual box size=0.02 0.02 0.02

Commit message: unstacking all towers working reasonably well

File: urdfs/objects/cube.urdf (robot description, URDF)
Before this commit: robot cube, 1 links, 0 joints
Links:
- link base_link: mass 1.2 -> 2
