Commit message: debugging ergo finger collision objects

File: urdfs/ergo_jr/poppy_ergo_jr.pybullet.urdf (robot description, URDF)
Before this commit: robot poppy_ergo_jr, 9 links, 8 joints
Links:
- link fixed_tip: geometry collision box size=0.020 0.030 0.05
- link section_5: geometry collision box size=0.0005 0.060 0.04

Commit message: t7f and t7m used for collision object placement, need to finalize t7m and move back to section 5 link

File: urdfs/ergo_jr/poppy_ergo_jr.pybullet.urdf (robot description, URDF)
Before this commit: robot poppy_ergo_jr, 9 links, 8 joints
Links:
- link fixed_tip: geometry collision box size=0.020 0.025 0.0005
- link moving_tip: geometry collision box size=0.0005 0.025 0.02
- link section_5: geometry visual mesh filename=meshes/gripper.stl
Joints:
- joint t7m: origin xyz=0 -0.052 0 rpy=-1.5707963267949 0 0 -> xyz=0 0 0 rpy=0 0 0

Commit message: finalized collision shapes and rough pickup working

File: urdfs/ergo_jr/poppy_ergo_jr.pybullet.urdf (robot description, URDF)
Before this commit: robot poppy_ergo_jr, 9 links, 8 joints
Links:
- link fixed_tip: geometry collision box size=0.020 0.025 0.003; visual box size=0 0 0
- link moving_tip: geometry collision box size=0.003 0.025 0.02; visual box size=0 0 0

Commit message: improved urdf for proper IK at fingertips

File: urdfs/ergo_jr/poppy_ergo_jr.pybullet.urdf (robot description, URDF)
Before this commit: robot poppy_ergo_jr, 9 links, 8 joints
Links:
- link base_link: geometry collision cylinder length=0.03 radius=0.08
- link fixed_tip: geometry collision box size=0.020 0.025 0.003
- link long_U: geometry collision cylinder length=0.02 radius=0.02
- link moving_tip: geometry collision box size=0.003 0.025 0.02
- link section_1: geometry collision cylinder length=0.05 radius=0.02
- link section_2: geometry collision cylinder length=0.05 radius=0.02
- link section_3: geometry collision cylinder length=0.05 radius=0.02
- link section_4: geometry collision cylinder length=0.03 radius=0.02; visual mesh filename=meshes/section_4.stl
Joints:
- joint t7f: origin xyz=0 -0.11 0 rpy=-1.5707963267949 0 0 -> xyz=0 -0.125 0.0155 rpy=0 0 0
- joint t7m: origin xyz=0 0 0 rpy=0 0 0 -> xyz=-0.0155 -0.0675 0 rpy=0 0 0

Commit message: added placeholder inertials to ergo_jr urdf to avoid b3 warnings

File: urdfs/ergo_jr/poppy_ergo_jr.pybullet.urdf (robot description, URDF)
Before this commit: robot poppy_ergo_jr, 9 links, 8 joints
Links:
- link base_link: mass None -> 1
- link fixed_tip: mass None -> 1
- link moving_tip: mass None -> 1

Commit message: dynamic duration in trajectories based on distance

File: urdfs/ergo_jr/poppy_ergo_jr.pybullet.urdf (robot description, URDF)
Before this commit: robot poppy_ergo_jr, 9 links, 8 joints
Links:
- link fixed_tip: mass 1 -> 1.0
