Commit message: made ergo forearms with help of openscad

File: urdfs/ergo/poppy_ergo.pybullet.urdf (robot description, URDF)
Before this commit: robot Poppy_Humanoid, 26 links, 25 joints
Links:
- link l_forearm: geometry collision mesh filename=meshes/l_forearm_respondable.STL; visual mesh filename=meshes/l_forearm_visual_ergo.STL
- link r_forearm: geometry collision mesh filename=meshes/r_forearm_respondable.STL; visual mesh filename=meshes/r_forearm_visual_ergo.STL

Commit message: added right gripper to ergo urdf

File: urdfs/ergo/poppy_ergo.pybullet.urdf (robot description, URDF)
Before this commit: robot Poppy_Humanoid, 26 links, 25 joints
Links:
- added link r_section_4, mass 0.1; collision cylinder length=0.03 radius=0.02; visual mesh filename=meshes/section_4.stl
- added link r_section_5, mass 0.1; visual mesh filename=meshes/gripper.stl
Joints:
- added joint m6: type continuous, parent r_section_4, child r_section_5, origin xyz=0 -0.058 0 rpy=0 -1.5707963267949 0, axis 0 0 -1
- added joint r_m5: type continuous, parent r_forearm, child r_section_4, origin xyz=-0.01 0.1 0 rpy=3.14159265358979 1.5707963267949 0, axis 0 0 1

File: urdfs/ergo_jr/poppy_ergo_jr.pybullet.urdf (robot description, URDF)
Before this commit: robot poppy_ergo_jr, 9 links, 8 joints
Links:
- link base_link: geometry collision cylinder length=0.03 radius=0.08; visual mesh filename=meshes/base.stl
- link fixed_tip: geometry collision box size=0.020 0.025 0.003; visual box size=0 0 0
- link long_U: geometry collision cylinder length=0.02 radius=0.02; visual mesh filename=meshes/long_U.stl
- link moving_tip: geometry collision box size=0.003 0.025 0.02; visual box size=0 0 0
- link section_1: geometry collision cylinder length=0.05 radius=0.02; visual mesh filename=meshes/section_1.stl
- link section_2: geometry collision cylinder length=0.05 radius=0.02; visual mesh filename=meshes/section_2.stl
- link section_3: geometry collision cylinder length=0.05 radius=0.02; visual mesh filename=meshes/section_3.stl

Commit message: started on more realistic ergo urdf

File: urdfs/ergo/poppy_ergo.pybullet.urdf (robot description, URDF)
Before this commit: robot Poppy_Humanoid, 28 links, 27 joints
Links:
- removed link r_section_4
- removed link r_section_5
- added link r_support_gripper, mass 0.1; collision cylinder length=0.03 radius=0.02; visual mesh filename=meshes/support_gripper.STL
Joints:
- removed joint m6
- removed joint r_m5
- added joint r_w: type fixed, parent r_forearm, child r_support_gripper, origin xyz=-0.01 0.1 0 rpy=3.14159265358979 1.5707963267949 0, axis 0 0 1

Commit message: more urdf progress

File: urdfs/ergo/poppy_ergo.pybullet.urdf (robot description, URDF)
Before this commit: robot Poppy_Humanoid, 27 links, 26 joints
Links:
- removed link r_support_gripper
- added link l_long_u, mass 0.1; collision cylinder length=0.03 radius=0.02; visual mesh filename=meshes/long_U.stl scale=1 1 1
- added link r_long_u, mass 0.1; collision cylinder length=0.03 radius=0.02; visual mesh filename=meshes/long_U.stl scale=1 1 1
- added link r_short_u, mass 0.1; collision cylinder length=0.03 radius=0.01; visual mesh filename=meshes/short_U.stl
- added link r_thumb, mass 0.1; visual mesh filename=meshes/gripper.stl
- link l_forearm: geometry collision mesh filename=meshes/l_forearm_respondable.STL; visual mesh filename=meshes/l_forearm_visual_ergo.STL
- link r_forearm: geometry collision mesh filename=meshes/r_forearm_respondable.STL; visual mesh filename=meshes/r_forearm_visual_ergo.STL
Joints:
- removed joint r_w
- added joint l_wrist_y: type revolute, parent l_forearm, child l_long_u, origin xyz=.01 .145 0 rpy=0 0 0, axis 0 1 0, limit lower=-3.14 upper=3.14 effort=3.1 velocity=7.0
- added joint r_gripper: type revolute, parent r_short_u, child r_thumb, origin xyz=0 -0.04 0 rpy=0 0 0, axis 0 0 1, limit lower=-3.14 upper=3.14 effort=3.1 velocity=7.0
- added joint r_wrist_x: type revolute, parent r_long_u, child r_short_u, origin xyz=0 0.025 0 rpy=0 0 0, axis 1 0 0, limit lower=-3.14 upper=3.14 effort=3.1 velocity=7.0
- added joint r_wrist_y: type revolute, parent r_forearm, child r_long_u, origin xyz=-.01 .145 0 rpy=0 0 0, axis 0 1 0, limit lower=-3.14 upper=3.14 effort=3.1 velocity=7.0

Commit message: finished visual shapes for each ergo hand

File: urdfs/ergo/poppy_ergo.pybullet.urdf (robot description, URDF)
Before this commit: robot Poppy_Humanoid, 30 links, 29 joints
Links:
- removed link r_short_u
- added link l_hand, mass 0.1; collision cylinder length=0.03 radius=0.01; visual mesh filename=meshes/gripper-fixed_part.stl scale=.001 .001 .001
- added link l_thumb, mass 0.1; visual mesh filename=meshes/gripper.stl
- added link r_hand, mass 0.1; collision cylinder length=0.03 radius=0.01; visual mesh filename=meshes/gripper-fixed_part.stl scale=.001 .001 .001
Joints:
- added joint l_gripper: type revolute, parent l_hand, child l_thumb, origin xyz=0 -0.04 0 rpy=0 1.5707963267949 0, axis 0 0 1, limit lower=-3.14 upper=3.14 effort=3.1 velocity=7.0
- added joint l_wrist_x: type revolute, parent l_long_u, child l_hand, origin xyz=0 0.025 0 rpy=0 0 0, axis 1 0 0, limit lower=-3.14 upper=3.14 effort=3.1 velocity=7.0
- joint r_gripper: origin xyz=0 -0.04 0 rpy=0 0 0 -> xyz=0 -0.04 0 rpy=0 1.5707963267949 0; parent r_short_u -> r_hand
- joint r_wrist_x: child r_short_u -> r_hand

Commit message: started motor shapes for each hand

File: urdfs/ergo/poppy_ergo.pybullet.urdf (robot description, URDF)
Before this commit: robot Poppy_Humanoid, 32 links, 31 joints
Links:
- link l_forearm: geometry collision mesh filename=meshes/l_forearm_respondable.STL; visual box size=0.025 0.0325 0.02
- link l_hand: geometry collision cylinder length=0.03 radius=0.01; visual box size=0.025 0.0325 0.02
- link r_forearm: geometry collision mesh filename=meshes/r_forearm_respondable.STL; visual box size=0.025 0.0325 0.02
- link r_hand: geometry collision cylinder length=0.03 radius=0.01; visual box size=0.025 0.0325 0.02

Commit message: finished motor shapes

File: urdfs/ergo/poppy_ergo.pybullet.urdf (robot description, URDF)
Before this commit: robot Poppy_Humanoid, 32 links, 31 joints
Links:
- link l_hand: geometry collision cylinder length=0.03 radius=0.01; visual box size=0.025 0.0325 0.02
- link r_hand: geometry collision cylinder length=0.03 radius=0.01; visual box size=0.025 0.0325 0.02

Commit message: finished collision shapes

File: urdfs/ergo/poppy_ergo.pybullet.urdf (robot description, URDF)
Before this commit: robot Poppy_Humanoid, 32 links, 31 joints
Links:
- added link l_fixed_tip, mass 1.0; collision box size=0.020 0.025 0.003; visual box size=0 0 0
- added link l_moving_tip, mass 1; collision box size=0.003 0.025 0.02; visual box size=0 0 0
- added link r_fixed_tip, mass 1.0; collision box size=0.020 0.025 0.003; visual box size=0 0 0
- added link r_moving_tip, mass 1; collision box size=0.003 0.025 0.02; visual box size=0 0 0
- link l_hand: geometry collision box size=0.025 0.0325 0.02; collision box size=0.025 0.035 0.02
- link l_long_u: geometry collision box size=0.03 0.0325 0.02; visual mesh filename=meshes/long_U.stl scale=1 1 1
- link r_hand: geometry collision box size=0.025 0.0325 0.02; collision box size=0.025 0.035 0.02
- link r_long_u: geometry collision box size=0.03 0.0325 0.02; visual mesh filename=meshes/long_U.stl scale=1 1 1
Joints:
- added joint l_fixed_tip: type fixed, parent l_hand, child l_fixed_tip, origin xyz=0 -0.11 -0.01325 rpy=0 0 0
- added joint l_moving_tip: type fixed, parent l_thumb, child l_moving_tip, origin xyz=-0.0155 -0.0675 0 rpy=0 0 0
- added joint r_fixed_tip: type fixed, parent r_hand, child r_fixed_tip, origin xyz=0 -0.11 -0.01325 rpy=0 0 0
- added joint r_moving_tip: type fixed, parent r_thumb, child r_moving_tip, origin xyz=-0.0155 -0.0675 0 rpy=0 0 0

Commit message: tweaked masses of hands (pybullet recomputes inertia matrix from collision shape)

File: urdfs/ergo/poppy_ergo.pybullet.urdf (robot description, URDF)
Before this commit: robot Poppy_Humanoid, 36 links, 35 joints
Links:
- link l_fixed_tip: mass 1.0 -> .01
- link l_hand: mass 0.1 -> 0.02
- link l_long_u: mass 0.1 -> 0.01
- link l_moving_tip: mass 1 -> .01
- link l_thumb: mass 0.1 -> 0.01
- link r_fixed_tip: mass 1.0 -> .01
- link r_hand: mass 0.1 -> 0.02
- link r_long_u: mass 0.1 -> 0.01
- link r_moving_tip: mass 1 -> .01
- link r_thumb: mass 0.1 -> 0.01
